File: iopcb.kicad_sch (KiCad schematic)
At the start: 21 parts, among them J1 Conn_01x03, J2 Conn_01x03, J3 Conn_01x03, J4 Conn_01x02, J5 Conn_01x02, J6 Conn_01x03, K1 EE2-24NU, U1 LM321

Commit message: updated
Parts:
- removed J1, J2, J3, J6: Conn_01x03, samsung_pcblib:15EDGRC-3.5-3P-PAK, symbol Connector_Generic:Conn_01x03
- removed J4, J5: Conn_01x02, samsung_pcblib:15EDGRC-3.5-2P-PAK, symbol Connector_Generic:Conn_01x02
- removed R4, R6, R8: 10K, Resistor_SMD:R_0603_1608Metric, symbol Device:R
- added C3: 10nF, Capacitor_SMD:C_0603_1608Metric, symbol Device:C
- added D2: 10V MM3Z10VC, Diode_SMD:D_SOD-323F, symbol Device:D_Zener
- added J1, J2: Conn_01x08, symbol Connector_Generic:Conn_01x08
- added JP1, JP2, JP3, JP4: SolderJumper_3_Open, TestPoint:TestPoint_2Pads_Pitch2.54mm_Drill0.8mm, symbol Jumper:SolderJumper_3_Open
- added R11: 1K, Resistor_SMD:R_0603_1608Metric, symbol Device:R
- R1: value 100K -> 30K
- renumbered D2 to D1, D1 to D3, R9 to R10, R5 to R8, R7 to R9
Connections:
- net +24V: now also J1.2 (Pin_2), JP1.1 (A), JP2.1 (A), JP3.1 (A), JP4.1 (A)
- net 1NO_Out: now also J2.1 (Pin_1), JP1.2 (C)
- net 2NO_Out: now also J2.3 (Pin_3), JP2.2 (C)
- net 3NO_Out: now also J2.5 (Pin_5), JP3.2 (C)
- net GND: now also D2.2 (A), J1.1 (Pin_1), JP1.3 (B), JP2.3 (B), JP3.3 (B), JP4.3 (B)
- net Safety_In: now also J1.6 (Pin_6)
- net Safety_OutA: now also J1.7 (Pin_7)
- net Safety_OutB: now also C3.2, J1.8 (Pin_8)
- net VBat_In: now also J1.4 (Pin_4)
- net VBat_Out: now also J1.5 (Pin_5)
- net at C1.1, R1.2, R2.1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: now also D2.1 (K)
- net 1NO_A renamed 1NO_In
- net 1NO_In: now also J2.2 (Pin_2)
- net 2NO_A renamed 2NO_In
- net 2NO_In: now also J2.4 (Pin_4)
- net 3NO_A renamed 3NO_In
- net 3NO_In: now also J2.6 (Pin_6)
- new net 4NO_In: J2.8 (Pin_8), R11.2
- new net 4NO_Out: J2.7 (Pin_7), JP4.2 (C), R11.1
Other:
- note added: "27K: Vmax 48V 30K: Vmax 54V 36K: Vmax 60V"
- note added: "4x Obsługa styków pomocniczych zabezpieczeń"
- note removed: "3x Obsługa styków pomocniczych zabezpieczeń"
- note removed: "Zasilanie płytki"
- moved on the sheet: C1, C2, D1, D3, K1, R1, R10, R2, R3, R9, U1
